File: Secondary/Secondary.kicad_pcb (KiCad board)
At the start: 4 copper layers, 78.4 x 61.5 mm, 14 parts, among them J3 Conn_01x05_Pin

Commit message: Added secondary clamp and swapped components
Parts:
- added IC9: BZX84-C5V6,215, BZX84-C5V6,215:SOT95P230X110-3N, F.Cu at (59.1, 132.0)
Routing:
- net GND_ISO: track 0.00 -> 19.3 mm, vias 0 -> 6
- net /IOUT_HIGH: track 43.0 -> 47.0 mm
Other:
- board text added: "tc"
