File: Secondary/Secondary.kicad_sch (KiCad schematic)
At the start: 14 parts, among them J3 Conn_01x05_Pin

Commit message: Added secondary clamp and swapped components
Parts:
- added IC9: BZX84-C5V6,215, BZX84-C5V6,215:SOT95P230X110-3N, symbol BZX84-C5V6_215:BZX84-C5V6,215
Connections:
- net GND_ISO: now also IC9.1 (A)
- net IOUT_HIGH: now also IC9.3 (K)
